File: FAMICOM_PROVE_CART.kicad_pcb (KiCad board)
At the start: 2 copper layers, 100 x 100 mm, 8 parts, among them J1 TEST1, J2 TEST2, J3 TEST3, J4 TEST4, U1 BUS_FC60, U2 BUS_FC60

Commit message: Rev 1.0 fix 1
Typo fix
Other:
- board text added: "FC TEST PROBE ADAPTER CARD REV0.1A Feb/2019 (C) @antarcticlion License: CC SA BY 4.0"
- board text removed: "FC TEST PROBE ADAPTER CARD REV0.1A Feb/2019 (C) @antarcticlion Licence: CC SA BY 4.0"
Changed lines of the file:
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@@
     )
   )
-  (gr_text "FC TEST PROBE ADAPTER CARD\nREV0.1A Feb/2019 (C) @antarcticlion\nLicence: CC SA BY 4.0" (at 66 80.5) (layer B.SilkS)
+  (gr_text "FC TEST PROBE ADAPTER CARD\nREV0.1A Feb/2019 (C) @antarcticlion\nLicense: CC SA BY 4.0" (at 66 80.5) (layer B.SilkS)
     (effects (font (size 1.5 1.5) (thickness 0.3)) (justify mirror))
   )
@@
   )
   (target plus (at 0 100) (size 5) (width 0.15) (layer Edge.Cuts))
-  (gr_text "FC TEST PROBE ADAPTER CARD\nREV0.1A Feb/2019 (C) @antarcticlion\nLicence: CC SA BY 4.0" (at 64 80.5) (layer F.SilkS)
+  (gr_text "FC TEST PROBE ADAPTER CARD\nREV0.1A Feb/2019 (C) @antarcticlion\nLicense: CC SA BY 4.0" (at 64 80.5) (layer F.SilkS)
     (effects (font (size 1.5 1.5) (thickness 0.3)))
   )
